File: sata-backplane.kicad_sch (KiCad schematic)
At the start: 26 parts, among them J5 457180002, J6 G40H3132212HR, U1 TPS563201DDCR, U5 TPS563201DDCR

Commit message: Routed
Connections:
- net S1_A+: now also J6.D4; no longer J6.C4
- net S1_A-: now also J6.D5; no longer J6.C5
- net S1_B+: now also J6.B4; no longer J6.A5
- net S1_B-: now also J6.B5; no longer J6.A4
- net S2_A+: now also J6.C4; no longer J6.D4
- net S2_A-: now also J6.C5; no longer J6.D5
- net S2_B+: now also J6.A4; no longer J6.D8
- net S2_B-: now also J6.A5; no longer J6.D7
- net S3_A+: now also J6.D7; no longer J6.C7
- net S3_A-: now also J6.D8; no longer J6.C8
- net S3_B+: now also J6.B7; no longer J6.A8
- net S3_B-: now also J6.B8; no longer J6.A7
- net S4_A+: now also J6.C7; no longer J6.B4
- net S4_A-: now also J6.C8; no longer J6.B5
- net S4_B+: now also J6.A7; no longer J6.B8
- net S4_B-: now also J6.A8; no longer J6.B7
Changed lines of the file:
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@@
 	)
 	(label "S3_A+"
-		(at 234.95 143.51 180)
-		(effects
-			(font
-				(size 1.27 1.27)
-			)
-			(justify right bottom)
+		(at 260.35 143.51 0)
+		(effects
+			(font
+				(size 1.27 1.27)
+			)
+			(justify left bottom)
 		)
 	)
 	(label "S4_B+"
-		(at 260.35 120.65 0)
-		(effects
-			(font
-				(size 1.27 1.27)
-			)
-			(justify left bottom)
+		(at 234.95 118.11 180)
+		(effects
+			(font
+				(size 1.27 1.27)
+			)
+			(justify right bottom)
 		)
 	)
@@
 	)
 	(label "S4_A-"
-		(at 260.35 113.03 0)
-		(effects
-			(font
-				(size 1.27 1.27)
-			)
-			(justify left bottom)
+		(at 234.95 146.05 180)
+		(effects
+			(font
+				(size 1.27 1.27)
+			)
+			(justify right bottom)
 		)
 	)
 	(label "S4_B-"
-		(at 260.35 118.11 0)
-		(effects
-			(font
-				(size 1.27 1.27)
-			)
-			(justify left bottom)
+		(at 234.95 120.65 180)
+		(effects
+			(font
+				(size 1.27 1.27)
+			)
+			(justify right bottom)
 		)
 	)
@@
 	)
 	(label "S1_B+"
-		(at 234.95 113.03 180)
-		(effects
-			(font
-				(size 1.27 1.27)
-			)
-			(justify right bottom)
+		(at 260.35 110.49 0)
+		(effects
+			(font
+				(size 1.27 1.27)
+			)
+			(justify left bottom)
 		)
 	)
 	(label "S3_A-"
-		(at 234.95 146.05 180)
-		(effects
-			(font
-				(size 1.27 1.27)
-			)
-			(justify right bottom)
+		(at 260.35 146.05 0)
+		(effects
+			(font
+				(size 1.27 1.27)
+			)
+			(justify left bottom)
 		)
 	)
@@
 	)
 	(label "S1_A-"
-		(at 234.95 138.43 180)
-		(effects
-			(font
-				(size 1.27 1.27)
-			)
-			(justify right bottom)
+		(at 260.35 138.43 0)
+		(effects
+			(font
+				(size 1.27 1.27)
+			)
+			(justify left bottom)
 		)
 	)
@@
 	)
 	(label "S4_A+"
-		(at 260.35 110.49 0)
-		(effects
-			(font
-				(size 1.27 1.27)
-			)
-			(justify left bottom)
+		(at 234.95 143.51 180)
+		(effects
+			(font
+				(size 1.27 1.27)
+			)
+			(justify right bottom)
 		)
 	)
@@
 	)
 	(label "S2_B+"
-		(at 260.35 146.05 0)
-		(effects
-			(font
-				(size 1.27 1.27)
-			)
-			(justify left bottom)
+		(at 234.95 110.49 180)
+		(effects
+			(font
+				(size 1.27 1.27)
+			)
+			(justify right bottom)
 		)
 	)
@@
 	)
 	(label "S1_B-"
-		(at 234.95 110.49 180)
-		(effects
-			(font
-				(size 1.27 1.27)
-			)
-			(justify right bottom)
+		(at 260.35 113.03 0)
+		(effects
+			(font
+				(size 1.27 1.27)
+			)
+			(justify left bottom)
 		)
 	)
@@
 	)
 	(label "S1_A+"
+		(at 260.35 135.89 0)
+		(effects
+			(font
+				(size 1.27 1.27)
+			)
+			(justify left bottom)
+		)
+	)
+	(label "S2_A+"
 		(at 234.95 135.89 180)
 		(effects
@@
 		)
 	)
-	(label "S2_A+"
-		(at 260.35 135.89 0)
-		(effects
-			(font
-				(size 1.27 1.27)
-			)
-			(justify left bottom)
-		)
-	)
 	(label "S3_B+"
-		(at 234.95 120.65 180)
-		(effects
-			(font
-				(size 1.27 1.27)
-			)
-			(justify right bottom)
+		(at 260.35 118.11 0)
+		(effects
+			(font
+				(size 1.27 1.27)
+			)
+			(justify left bottom)
 		)
 	)
 	(label "S3_B-"
-		(at 234.95 118.11 180)
-		(effects
-			(font
-				(size 1.27 1.27)
-			)
-			(justify right bottom)
+		(at 260.35 120.65 0)
+		(effects
+			(font
+				(size 1.27 1.27)
+			)
+			(justify left bottom)
 		)
 	)
 	(label "S2_B-"
-		(at 260.35 143.51 0)
-		(effects
-			(font
-				(size 1.27 1.27)
-			)
-			(justify left bottom)
+		(at 234.95 113.03 180)
+		(effects
+			(font
+				(size 1.27 1.27)
+			)
+			(justify right bottom)
 		)
 	)
@@
 	)
 	(label "S2_A-"
-		(at 260.35 138.43 0)
-		(effects
-			(font
-				(size 1.27 1.27)
-			)
-			(justify left bottom)
-		)
-	)
+		(at 234.95 138.43 180)
+		(effects
+			(font
+				(size 1.27 1.27)
+			)
+			(justify right bottom)
+		)
+	)

Commit message: Add Molex HD power connector
Parts:
- added J7: Conn_01x04, 00-Local:350211-1_TYC, symbol Connector_Generic:Conn_01x04
- added JP1, JP2: SolderJumper_3_Open, Jumper:SolderJumper-3_P1.3mm_Bridged12_RoundedPad1.0x1.5mm, symbol Jumper:SolderJumper_3_Bridged12
- J5: footprint 00_Local:CONN_SD-45718-001_MOL -> 00-Local:CONN_SD-45718-001_MOL
Connections:
- net +12V: now also J7.1 (Pin_1)
- net +5V_1: now also JP1.2 (C); no longer C18.2, L5.2, R10.2
- net +5V_2: now also JP2.2 (C); no longer C4.2, L1.2, R2.2
- net GND: now also J7.2 (Pin_2), J7.3 (Pin_3)
- new net +5V: J7.4 (Pin_4), JP1.1 (A), JP2.1 (A)
- new net Converter1: C18.2, JP1.3 (B), L5.2, R10.2
- new net Converter2: C4.2, JP2.3 (B), L1.2, R2.2
Other:
- note added: "4 pin, 5.08mm pitch AMP Mate-N-Lok Molex 8981 C706976 C492551 C492552 C706975"
- note added: "External 5V"
- note added: "Onboard Converter"
- note added: "SATA 1/2"
- note added: "SATA 3/4"
